File: flashlight-stm32-dev/flashlight-stm32-dev.kicad_pcb (KiCad board)
At the start: 6 copper layers, 120 x 35 mm, 88 parts, among them J1 USB_C_Receptacle, J2 ST-LINK, Q1 2N7002H, Q2 2N7002H, Q3 2N7002H, SW1 RESET, SW2 BOOT, U1 BQ25185DLHR, U2 STM32L151C8Tx, U3 BMA400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

Commit message: with headers
Parts:
- added J3: IO1, Connector_PinHeader_2.54mm:PinHeader_1x11_P2.54mm_Vertical, F.Cu at (153.3, 145.0)
- added J4: IO2, Connector_PinHeader_2.54mm:PinHeader_1x11_P2.54mm_Vertical, F.Cu at (153.3, 114.0)
- added JP1: Jumper_2_Bridged, Jumper:SolderJumper-2_P1.3mm_Bridged_RoundedPad1.0x1.5mm, F.Cu at (157.9, 138.7)
- moved D3 0.25 mm to (100.8, 137.7)
Connections:
- U2 pad 11: unconnected-(U2-PA1-Pad11) -> /PA1
- U2 pad 12: unconnected-(U2-PA2-Pad12) -> /PA2
- U2 pad 13: unconnected-(U2-PA3-Pad13) -> /PA3
- U2 pad 14: unconnected-(U2-PA4-Pad14) -> /PA4
- U2 pad 15: unconnected-(U2-PA5-Pad15) -> /PA5
- U2 pad 16: unconnected-(U2-PA6-Pad16) -> /PA6
- U2 pad 17: unconnected-(U2-PA7-Pad17) -> /PA7
- U2 pad 21: unconnected-(U2-PB10-Pad21) -> /PB10
- U2 pad 22: unconnected-(U2-PB11-Pad22) -> /PB11
- U2 pad 25: unconnected-(U2-PB12-Pad25) -> /PB12
- U2 pad 26: unconnected-(U2-PB13-Pad26) -> /PB13
- U2 pad 27: unconnected-(U2-PB14-Pad27) -> /PB14
- U2 pad 28: unconnected-(U2-PB15-Pad28) -> /PB15
- U2 pad 29: unconnected-(U2-PA8-Pad29) -> /PA8
- U2 pad 30: unconnected-(U2-PA9-Pad30) -> /PA9
- U2 pad 31: unconnected-(U2-PA10-Pad31) -> /PA10
- U2 pad 38: unconnected-(U2-PA15-Pad38) -> /PA15
- U2 pad 39: unconnected-(U2-PB3-Pad39) -> /PB3
Routing:
- net /PA10: track 0.00 -> 34.4 mm, vias 0 -> 1
- net /PA9: track 0.00 -> 33.5 mm, vias 0 -> 1
- net /PA8: track 0.00 -> 32.5 mm, vias 0 -> 1
- net /PB15: track 0.00 -> 31.2 mm, vias 0 -> 1
- net /PB14: track 0.00 -> 29.9 mm, vias 0 -> 1
- net /PB13: track 0.00 -> 28.5 mm, vias 0 -> 1
- net /PB12: track 0.00 -> 27.1 mm, vias 0 -> 1
- net /PA2: track 0.00 -> 23.3 mm, vias 0 -> 1
- net /PB3: track 0.00 -> 18.6 mm
- net /PA1: track 0.00 -> 18.5 mm, vias 0 -> 1
- net /PA15: track 0.00 -> 16.5 mm
- net /PB11: track 0.00 -> 14.9 mm
- net /PA3: track 0.00 -> 14.3 mm
- net /PB10: track 0.00 -> 13.1 mm
- net /PA7: track 0.00 -> 12.9 mm
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- added copper zone on In4.Cu, net /BAT+
