File: flashlight-stm32-dev/flashlight-stm32-dev.kicad_sch (KiCad schematic)
At the start: 99 parts, among them J1 USB_C_Receptacle, J2 ST-LINK, J3 IO1, J4 IO2, Q1 2N7002H, Q2 2N7002H, Q3 2N7002H, SW1 RESET, SW2 BOOT, U1 BQ25185DLHR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

Commit message: updates
Parts:
- removed RU22: 0, Resistor_SMD:R_0603_1608Metric_Pad0.98x0.95mm_HandSolder, symbol Device:R_US
- added CU210: 100n, Capacitor_SMD:C_0603_1608Metric_Pad1.08x0.95mm_HandSolder, symbol Device:C_Small
- D1: footprint LED_THT:LED_D5.0mm-4_RGB_Staggered_Pins -> 19-237_R6GHBHC-A01_2T:19237R6GHBHCA012T; symbol Device:LED_BARG -> Device:LED_RGBA
- J3, J4: footprint Connector_PinHeader_2.54mm:PinHeader_1x11_P2.54mm_Vertical -> Connector_PinHeader_2.54mm:PinHeader_1x12_P2.54mm_Vertical; symbol Connector:Conn_01x11_Pin -> Connector:Conn_01x12_Pin
Connections:
- net +3.3V: now also D1.4 (A), J3.11 (Pin_11), J4.2 (Pin_2); no longer D1.2 (A), J3.10 (Pin_10), J4.1 (Pin_1)
- net GND: now also J3.1 (Pin_1), J3.12 (Pin_12), J4.3 (Pin_3), CU210.2; no longer J3.11 (Pin_11), J4.2 (Pin_2)
- net PA1: now also J3.2 (Pin_2); no longer J3.1 (Pin_1)
- net PA10: now also J4.6 (Pin_6); no longer J4.5 (Pin_5)
- net PA15: now also J4.5 (Pin_5); no longer J4.4 (Pin_4)
- net PA2: now also J3.3 (Pin_3); no longer J3.2 (Pin_2)
- net PA3: now also J3.4 (Pin_4); no longer J3.3 (Pin_3)
- net PA4: now also J3.5 (Pin_5); no longer J3.4 (Pin_4)
- net PA5: now also J3.6 (Pin_6); no longer J3.5 (Pin_5)
- net PA6: now also J3.7 (Pin_7); no longer J3.6 (Pin_6)
- net PA7: now also J3.8 (Pin_8); no longer J3.7 (Pin_7)
- net PA8: now also J4.8 (Pin_8); no longer J4.7 (Pin_7)
- net PA9: now also J4.7 (Pin_7); no longer J4.6 (Pin_6)
- net PB10: now also J3.9 (Pin_9); no longer J3.8 (Pin_8)
- net PB11: now also J3.10 (Pin_10); no longer J3.9 (Pin_9)
- net PB12: now also J4.12 (Pin_12); no longer J4.11 (Pin_11)
- net PB13: now also J4.11 (Pin_11); no longer J4.10 (Pin_10)
- net PB14: now also J4.10 (Pin_10); no longer J4.9 (Pin_9)
- net PB15: now also J4.9 (Pin_9); no longer J4.8 (Pin_8)
- net PB3: now also J4.4 (Pin_4); no longer J4.3 (Pin_3)
- net at RD11.2: now also D1.1 (RK); no longer D1.3 (RK)
- net VLCD: now reaches U2.1 (VLCD)
- net VLCD: now also J4.1 (Pin_1), CU210.1
- net at RD12.2: now also D1.2 (GK); no longer D1.4 (GK)
- net at RD13.2: now also D1.3 (BK); no longer D1.1 (BK)
