File: flashlight-full-v1/flashlight-full-v1.kicad_pcb (KiCad board)
At the start: 6 copper layers, 120 x 35 mm, 99 parts, among them J1 USB_C_Receptacle, J2 ST-LINK, J3 IO1, J4 IO2, J5 SYS, J6 GND, Q1 2N7002H, Q2 2N7002H, Q3 2N7002H, SW1 RESET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

Commit message: full init
Changed lines of the file:
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@@
 		(at 100.965 92.8624)
 		(property "Reference" "U6"
-			(at 0.254 2.3876 180)
+			(at 2.9464 1.1938 180)
 			(layer "F.SilkS")
 			(effects
