File: flashlight-led/flashlight-led.kicad_pcb (KiCad board)
At the start: 2 copper layers, 35 x 35 mm, 10 parts, among them J1 +18V, J2 GND, J3 GND

Commit message: full init
Parts:
- removed J2: GND, TestPoint:TestPoint_THTPad_D3.0mm_Drill1.5mm
- moved J3 18.5 mm to (164.7, 94.9)
- moved J1 13.0 mm to (157.8, 94.9)
- turned D1 to -90 degrees
- turned D2 to -150 degrees
- turned D3 to 150 degrees
Other:
- board size 35 x 35 mm -> 32 x 32 mm
